File: pcb/esp_all2.brd (EAGLE design)
At the start: 45 x 95 mm, 22 parts

Commit message: Improved ESP readability
Connections:
- net N$17 renamed DIMMING
Changed lines of the file:
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@@
 <?xml version="1.0" encoding="utf-8"?>
 <!DOCTYPE eagle SYSTEM "eagle.dtd">
-<eagle version="7.7.0">
+<eagle version="7.6.0">
 <drawing>
 <settings>
@@
 <wire x1="23.3" y1="58.1" x2="20" y2="61.4" width="1.27" layer="16"/>
 </signal>
-<signal name="N$17">
+<signal name="DIMMING">
 <contactref element="DIMMING" pad="4"/>
 <contactref element="DIMMING" pad="2"/>
