File: pcb/ads1115/ads1115_2.brd (EAGLE design)
At the start: 91.1 x 50 mm, 64 parts

Commit message: added resisitor values to schematic
Parts:
- R1, R10, R11, R12, R13, R14, R15, R16, R17, R18, R4, R5, R6, R7, R8, R9: value 4.7k -> 100R
- R19, R20, R21, R22, R23, R24, R25, R26, R27, R28, R29, R30, R31, R32, R33, R34: value 4.7k -> 1k
- R35, R36, R37, R38, R39, R40, R41, R42: value 4.7k -> n.a.
