File: pcb/ads1115/ads1115_2.sch (EAGLE design)
At the start: 64 parts

Commit message: added resisitor values to schematic
Parts:
- R1, R10, R11, R12, R13, R14, R15, R16, R17, R18, R4, R5, R6, R7, R8, R9: value 4.7k -> 100R
- R19, R20, R21, R22, R23, R24, R25, R26, R27, R28, R29, R30, R31, R32, R33, R34: value 4.7k -> 1k
- R35, R36, R37, R38, R39, R40, R41, R42: value 4.7k -> n.a.
Changed lines of the file:
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@@
 <part name="GND7" library="supply1" deviceset="GND" device=""/>
 <part name="P+7" library="supply1" deviceset="VCC" device=""/>
-<part name="R1" library="rcl" deviceset="R-EU_" device="M0805" value="4.7k"/>
-<part name="R4" library="rcl" deviceset="R-EU_" device="M0805" value="4.7k"/>
-<part name="R5" library="rcl" deviceset="R-EU_" device="M0805" value="4.7k"/>
-<part name="R6" library="rcl" deviceset="R-EU_" device="M0805" value="4.7k"/>
-<part name="R7" library="rcl" deviceset="R-EU_" device="M0805" value="4.7k"/>
-<part name="R8" library="rcl" deviceset="R-EU_" device="M0805" value="4.7k"/>
-<part name="R9" library="rcl" deviceset="R-EU_" device="M0805" value="4.7k"/>
-<part name="R10" library="rcl" deviceset="R-EU_" device="M0805" value="4.7k"/>
-<part name="R11" library="rcl" deviceset="R-EU_" device="M0805" value="4.7k"/>
-<part name="R12" library="rcl" deviceset="R-EU_" device="M0805" value="4.7k"/>
-<part name="R13" library="rcl" deviceset="R-EU_" device="M0805" value="4.7k"/>
-<part name="R14" library="rcl" deviceset="R-EU_" device="M0805" value="4.7k"/>
-<part name="R15" library="rcl" deviceset="R-EU_" device="M0805" value="4.7k"/>
-<part name="R16" library="rcl" deviceset="R-EU_" device="M0805" value="4.7k"/>
-<part name="R17" library="rcl" deviceset="R-EU_" device="M0805" value="4.7k"/>
-<part name="R18" library="rcl" deviceset="R-EU_" device="M0805" value="4.7k"/>
+<part name="R1" library="rcl" deviceset="R-EU_" device="M0805" value="100R"/>
+<part name="R4" library="rcl" deviceset="R-EU_" device="M0805" value="100R"/>
+<part name="R5" library="rcl" deviceset="R-EU_" device="M0805" value="100R"/>
+<part name="R6" library="rcl" deviceset="R-EU_" device="M0805" value="100R"/>
+<part name="R7" library="rcl" deviceset="R-EU_" device="M0805" value="100R"/>
+<part name="R8" library="rcl" deviceset="R-EU_" device="M0805" value="100R"/>
+<part name="R9" library="rcl" deviceset="R-EU_" device="M0805" value="100R"/>
+<part name="R10" library="rcl" deviceset="R-EU_" device="M0805" value="100R"/>
+<part name="R11" library="rcl" deviceset="R-EU_" device="M0805" value="100R"/>
+<part name="R12" library="rcl" deviceset="R-EU_" device="M0805" value="100R"/>
+<part name="R13" library="rcl" deviceset="R-EU_" device="M0805" value="100R"/>
+<part name="R14" library="rcl" deviceset="R-EU_" device="M0805" value="100R"/>
+<part name="R15" library="rcl" deviceset="R-EU_" device="M0805" value="100R"/>
+<part name="R16" library="rcl" deviceset="R-EU_" device="M0805" value="100R"/>
+<part name="R17" library="rcl" deviceset="R-EU_" device="M0805" value="100R"/>
+<part name="R18" library="rcl" deviceset="R-EU_" device="M0805" value="100R"/>
 <part name="U$16" library="JKW_CHIP" deviceset="2_PIN_CONNECTOR" device="" value="V1"/>
 <part name="U$17" library="JKW_CHIP" deviceset="2_PIN_CONNECTOR" device="" value="V1"/>
@@
 <part name="U$20" library="JKW_CHIP" deviceset="2_PIN_CONNECTOR" device="" value="V1"/>
 <part name="SV1" library="con-lstb" deviceset="MA04-1" device=""/>
-<part name="R19" library="rcl" deviceset="R-EU_" device="M0805" value="4.7k"/>
-<part name="R20" library="rcl" deviceset="R-EU_" device="M0805" value="4.7k"/>
-<part name="R21" library="rcl" deviceset="R-EU_" device="M0805" value="4.7k"/>
-<part name="R22" library="rcl" deviceset="R-EU_" device="M0805" value="4.7k"/>
-<part name="R23" library="rcl" deviceset="R-EU_" device="M0805" value="4.7k"/>
-<part name="R24" library="rcl" deviceset="R-EU_" device="M0805" value="4.7k"/>
-<part name="R25" library="rcl" deviceset="R-EU_" device="M0805" value="4.7k"/>
-<part name="R26" library="rcl" deviceset="R-EU_" device="M0805" value="4.7k"/>
-<part name="R27" library="rcl" deviceset="R-EU_" device="M0805" value="4.7k"/>
-<part name="R28" library="rcl" deviceset="R-EU_" device="M0805" value="4.7k"/>
-<part name="R29" library="rcl" deviceset="R-EU_" device="M0805" value="4.7k"/>
-<part name="R30" library="rcl" deviceset="R-EU_" device="M0805" value="4.7k"/>
-<part name="R31" library="rcl" deviceset="R-EU_" device="M0805" value="4.7k"/>
-<part name="R32" library="rcl" deviceset="R-EU_" device="M0805" value="4.7k"/>
-<part name="R33" library="rcl" deviceset="R-EU_" device="M0805" value="4.7k"/>
-<part name="R34" library="rcl" deviceset="R-EU_" device="M0805" value="4.7k"/>
-<part name="R35" library="rcl" deviceset="R-EU_" device="M0805" value="4.7k"/>
-<part name="R36" library="rcl" deviceset="R-EU_" device="M0805" value="4.7k"/>
-<part name="R37" library="rcl" deviceset="R-EU_" device="M0805" value="4.7k"/>
-<part name="R38" library="rcl" deviceset="R-EU_" device="M0805" value="4.7k"/>
-<part name="R39" library="rcl" deviceset="R-EU_" device="M0805" value="4.7k"/>
-<part name="R40" library="rcl" deviceset="R-EU_" device="M0805" value="4.7k"/>
-<part name="R41" library="rcl" deviceset="R-EU_" device="M0805" value="4.7k"/>
-<part name="R42" library="rcl" deviceset="R-EU_" device="M0805" value="4.7k"/>
+<part name="R19" library="rcl" deviceset="R-EU_" device="M0805" value="1k"/>
+<part name="R20" library="rcl" deviceset="R-EU_" device="M0805" value="1k"/>
+<part name="R21" library="rcl" deviceset="R-EU_" device="M0805" value="1k"/>
+<part name="R22" library="rcl" deviceset="R-EU_" device="M0805" value="1k"/>
+<part name="R23" library="rcl" deviceset="R-EU_" device="M0805" value="1k"/>
+<part name="R24" library="rcl" deviceset="R-EU_" device="M0805" value="1k"/>
+<part name="R25" library="rcl" deviceset="R-EU_" device="M0805" value="1k"/>
+<part name="R26" library="rcl" deviceset="R-EU_" device="M0805" value="1k"/>
+<part name="R27" library="rcl" deviceset="R-EU_" device="M0805" value="1k"/>
+<part name="R28" library="rcl" deviceset="R-EU_" device="M0805" value="1k"/>
+<part name="R29" library="rcl" deviceset="R-EU_" device="M0805" value="1k"/>
+<part name="R30" library="rcl" deviceset="R-EU_" device="M0805" value="1k"/>
+<part name="R31" library="rcl" deviceset="R-EU_" device="M0805" value="1k"/>
+<part name="R32" library="rcl" deviceset="R-EU_" device="M0805" value="1k"/>
+<part name="R33" library="rcl" deviceset="R-EU_" device="M0805" value="1k"/>
+<part name="R34" library="rcl" deviceset="R-EU_" device="M0805" value="1k"/>
+<part name="R35" library="rcl" deviceset="R-EU_" device="M0805" value="n.a."/>
+<part name="R36" library="rcl" deviceset="R-EU_" device="M0805" value="n.a."/>
+<part name="R37" library="rcl" deviceset="R-EU_" device="M0805" value="n.a."/>
+<part name="R38" library="rcl" deviceset="R-EU_" device="M0805" value="n.a."/>
+<part name="R39" library="rcl" deviceset="R-EU_" device="M0805" value="n.a."/>
+<part name="R40" library="rcl" deviceset="R-EU_" device="M0805" value="n.a."/>
+<part name="R41" library="rcl" deviceset="R-EU_" device="M0805" value="n.a."/>
+<part name="R42" library="rcl" deviceset="R-EU_" device="M0805" value="n.a."/>
 </parts>
 <sheets>
